File: v0/v0.kicad_pcb (KiCad board)
At the start: 2 copper layers, 101.5 x 88.1 mm, 40 parts, among them CON1 SNES-CONN, U1 SN74LV165APWR, U2 SN74LV165APWR, U3 SN74LV165APWR, U4 SN74LVC8T245PWR, U5 PIC12F629-ISN, U6 AMS1117-3.3, U7 SN74LVC8T245PWR, U8 Pico

Commit message: Critical fix to PSRAM to control /CE pin from Pico; add LCSC properties to all parts; add ICSP header for PIC12F
Parts:
- added ICSP1: Conn_01x05, Connector_PinHeader_2.54mm:PinHeader_1x05_P2.54mm_Vertical, F.Cu at (171.7, 96.5)
- added M1: LY68L6400SLIT, Package_SO:SOIC-8_3.9x4.9mm_P1.27mm, B.Cu at (115.4, 69.8)
- added R3: 10kR, Resistor_SMD:R_1206_3216Metric_Pad1.30x1.75mm_HandSolder, F.Cu at (172.9, 100.0)
- RN1, RN10, RN12, RN13, RN14, RN2, RN3, RN4, RN5, RN6, RN7, RN8: value R_Pack04 -> 100R
- U5: value PIC12F629-ISN -> PIC12F629-I/SN
- U8: value Pico -> Pair of 20-pin 1.27mm pitch vertical pin headers
Connections:
- U5 pad 4: unconnected-(U5-Pad4) -> /ICSPVPP
- U8 pad 27: unconnected-(U8-Pad27) -> /PSRAM_SIO0
- U8 pad 29: unconnected-(U8-Pad29) -> /PSRAM_SIO1
- U8 pad 31: unconnected-(U8-Pad31) -> /PSRAM_SIO2
- U8 pad 32: unconnected-(U8-Pad32) -> /PSRAM_SIO3
- U8 pad 33: unconnected-(U8-Pad33) -> GND
- U8 pad 34: unconnected-(U8-Pad34) -> /PSRAM_~{CE}
Routing:
- net +3.3V: track 137.8 -> 183.1 mm, vias 3 -> 4
- net /CLK_133MHZ: track 37.2 -> 72.6 mm, vias 3 -> 4
- net /ICSPVPP: track 0.00 -> 22.5 mm, vias 0 -> 2
- net /PSRAM_SIO0: track 0.00 -> 19.2 mm
- net /PSRAM_SIO1: track 0.00 -> 18.9 mm
- net /PSRAM_SIO3: track 0.00 -> 16.0 mm
- net /CIC_OUT: track 36.2 -> 51.8 mm
- net /CIC_IN: track 27.6 -> 42.2 mm
- net /PSRAM_~{CE}: track 0.00 -> 12.6 mm
- net /PSRAM_SIO2: track 0.00 -> 10.5 mm
- net GND: track 20.7 -> 28.2 mm, vias 8 -> 7
- net +5V: track 155.3 -> 160.8 mm
