File: v0/v0.kicad_sch (KiCad schematic)
At the start: 43 parts, among them CON1 SNES-CONN, M1 LY68L6400SLIT, U1 SN74LV165APWR, U2 SN74LV165APWR, U3 SN74LV165APWR, U4 SN74LVC8T245PWR, U5 PIC12F629-I/SN, U6 AMS1117-3.3, U7 SN74LVC8T245PWR, U8 Pair of 20-pin 1.27mm pitch v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

Commit message: Add LCSC and MOUSER part numbers
Parts:
- C1, C10, C12, C13, C14, C2, C3, C4, C5, C7: LCSC (none) -> C110255; MOUSER (none) -> 80-C1206C104K5R7210
- C11, C9: LCSC (none) -> C9807; MOUSER (none) -> 187-CL31B106KQHNFNE
- C15, C6, C8: LCSC (none) -> C444884; MOUSER (none) -> 187-CL31B105KAHNFNE
- ICSP1: MOUSER (none) -> 649-1012937890501BLF
- M1: MOUSER (none) -> 878-APS6404L-3SQN-SN
- R1, R2: LCSC (none) -> C113307; MOUSER (none) -> 660-RK73B2BTTDD101J
- R3: LCSC (none) -> C136460; MOUSER (none) -> CR1206-JW-103ELF
- RN1, RN10, RN11, RN12, RN13, RN14, RN2, RN3, RN4, RN5, RN6, RN7, RN8, RN9: MOUSER (none) -> 652-CAT16-101J4LF
- U1, U2, U3: MOUSER (none) -> 595-SN74LV166APWR
- U4, U7: MOUSER (none) -> 595-SN74LVC8T245PWR
- U5: MOUSER (none) -> 579-PIC12F752-I/SN
- U6: MOUSER (none) -> 926-LM1117MPX3.3NOPB
- U8: LCSC (none) -> C3408; MOUSER (none) -> 855-M50-3532042
