File: v1/v1.kicad_sch (KiCad schematic)
At the start: 62 parts, among them CON1 SNES-CONN

Commit message: v1: switched back to TSSOP-16 package shift register for better switching characteristics; routed entire pcb
Parts:
- ADDR1, ADDR2, ADDR3, ADDR4: value 74LV165D,118 -> SN74LV165APWR; footprint Package_SO:SOIC-16_3.9x9.9mm_P1.27mm -> Package_SO:TSSOP-16_4.4x5mm_P0.65mm; LCSC C547919 -> C201716
- SRAM1: LCSC LY68L6400SLIT -> C261881
Connections:
- net CLK_INH renamed ~{ADDRCE}
Changed lines of the file:
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@@
     (effects (font (size 1.27 1.27)) (justify right bottom))
   )
-  (label "CLK_INH" (at 63.5 67.31 180)
+  (label "~{ADDRCE}" (at 63.5 67.31 180)
     (effects (font (size 1.27 1.27)) (justify right bottom))
   )
@@
     (effects (font (size 1.27 1.27)) (justify right bottom))
   )
-  (label "CLK_INH" (at 173.99 152.4 0)
+  (label "~{ADDRCE}" (at 173.99 152.4 0)
     (effects (font (size 1.27 1.27)) (justify left bottom))
   )
@@
     (effects (font (size 1.27 1.27)) (justify right bottom))
   )
-  (label "CLK_INH" (at 25.4 67.31 180)
+  (label "~{ADDRCE}" (at 25.4 67.31 180)
     (effects (font (size 1.27 1.27)) (justify right bottom))
   )
@@
     (effects (font (size 1.27 1.27)) (justify left bottom))
   )
-  (label "CLK_INH" (at 101.6 67.31 180)
+  (label "~{ADDRCE}" (at 101.6 67.31 180)
     (effects (font (size 1.27 1.27)) (justify right bottom))
   )
@@
     (effects (font (size 1.27 1.27)) (justify right bottom))
   )
-  (label "CLK_INH" (at 139.7 67.31 180)
+  (label "~{ADDRCE}" (at 139.7 67.31 180)
     (effects (font (size 1.27 1.27)) (justify right bottom))
   )
@@
     (in_bom yes) (on_board yes)
     (property "Reference" "ADDR4" (id 0) (at 152.4 48.26 0))
-    (property "Value" "74LV165D,118" (id 1) (at 152.4 50.8 0))
-    (property "Footprint" "Package_SO:SOIC-16_3.9x9.9mm_P1.27mm" (id 2) (at 152.4 49.53 0)
+    (property "Value" "SN74LV165APWR" (id 1) (at 158.75 60.96 90))
+    (property "Footprint" "Package_SO:TSSOP-16_4.4x5mm_P0.65mm" (id 2) (at 152.4 49.53 0)
       (effects (font (size 1.27 1.27)) hide)
     )
-    (property "Datasheet" "https://datasheet.lcsc.com/lcsc/2007030014_Nexperia-74LV165D-118_C547919.pdf" (id 3) (at 152.4 49.53 0)
+    (property "Datasheet" "https://www.ti.com/cn/lit/ds/symlink/sn74lv165a.pdf" (id 3) (at 152.4 49.53 0)
       (effects (font (size 1.27 1.27)) hide)
     )
-    (property "LCSC" "C547919" (id 4) (at 152.4 49.53 0)
+    (property "LCSC" "C201716" (id 4) (at 152.4 49.53 0)
       (effects (font (size 1.27 1.27)) hide)
     )
@@
     (in_bom yes) (on_board yes)
     (property "Reference" "ADDR1" (id 0) (at 38.1 48.26 0))
-    (property "Value" "74LV165D,118" (id 1) (at 38.1 50.8 0))
-    (property "Footprint" "Package_SO:SOIC-16_3.9x9.9mm_P1.27mm" (id 2) (at 38.1 49.53 0)
+    (property "Value" "SN74LV165APWR" (id 1) (at 44.45 60.96 90))
+    (property "Footprint" "Package_SO:TSSOP-16_4.4x5mm_P0.65mm" (id 2) (at 38.1 49.53 0)
       (effects (font (size 1.27 1.27)) hide)
     )
-    (property "Datasheet" "https://datasheet.lcsc.com/lcsc/2007030014_Nexperia-74LV165D-118_C547919.pdf" (id 3) (at 38.1 49.53 0)
+    (property "Datasheet" "https://www.ti.com/cn/lit/ds/symlink/sn74lv165a.pdf" (id 3) (at 38.1 49.53 0)
       (effects (font (size 1.27 1.27)) hide)
     )
-    (property "LCSC" "C547919" (id 4) (at 38.1 49.53 0)
+    (property "LCSC" "C201716" (id 4) (at 38.1 49.53 0)
       (effects (font (size 1.27 1.27)) hide)
     )
@@
     (in_bom yes) (on_board yes)
     (property "Reference" "ADDR3" (id 0) (at 114.3 48.26 0))
-    (property "Value" "74LV165D,118" (id 1) (at 114.3 50.8 0))
-    (property "Footprint" "Package_SO:SOIC-16_3.9x9.9mm_P1.27mm" (id 2) (at 114.3 49.53 0)
+    (property "Value" "SN74LV165APWR" (id 1) (at 120.65 60.96 90))
+    (property "Footprint" "Package_SO:TSSOP-16_4.4x5mm_P0.65mm" (id 2) (at 114.3 49.53 0)
       (effects (font (size 1.27 1.27)) hide)
     )
-    (property "Datasheet" "https://datasheet.lcsc.com/lcsc/2007030014_Nexperia-74LV165D-118_C547919.pdf" (id 3) (at 114.3 49.53 0)
+    (property "Datasheet" "https://www.ti.com/cn/lit/ds/symlink/sn74lv165a.pdf" (id 3) (at 114.3 49.53 0)
       (effects (font (size 1.27 1.27)) hide)
     )
-    (property "LCSC" "C547919" (id 4) (at 114.3 49.53 0)
+    (property "LCSC" "C201716" (id 4) (at 114.3 49.53 0)
       (effects (font (size 1.27 1.27)) hide)
     )
@@
     (in_bom yes) (on_board yes)
     (property "Reference" "ADDR2" (id 0) (at 76.2 48.26 0))
-    (property "Value" "74LV165D,118" (id 1) (at 76.2 50.8 0))
-    (property "Footprint" "Package_SO:SOIC-16_3.9x9.9mm_P1.27mm" (id 2) (at 76.2 49.53 0)
+    (property "Value" "SN74LV165APWR" (id 1) (at 82.55 60.96 90))
+    (property "Footprint" "Package_SO:TSSOP-16_4.4x5mm_P0.65mm" (id 2) (at 76.2 49.53 0)
       (effects (font (size 1.27 1.27)) hide)
     )
-    (property "Datasheet" "https://assets.nexperia.com/documents/data-sheet/74HC_HCT165.pdf" (id 3) (at 76.2 49.53 0)
+    (property "Datasheet" "https://www.ti.com/cn/lit/ds/symlink/sn74lv165a.pdf" (id 3) (at 76.2 49.53 0)
       (effects (font (size 1.27 1.27)) hide)
     )
-    (property "LCSC" "C547919" (id 4) (at 76.2 49.53 0)
+    (property "LCSC" "C201716" (id 4) (at 76.2 49.53 0)
       (effects (font (size 1.27 1.27)) hide)
     )
@@
       (effects (font (size 1.27 1.27)) hide)
     )
-    (property "LCSC" "LY68L6400SLIT" (id 4) (at 157.48 186.69 90)
+    (property "LCSC" "C261881" (id 4) (at 157.48 186.69 90)
       (effects (font (size 1.27 1.27)) hide)
     )
@@
     )
     (path "/3996c8d9-362a-4ae0-9ed6-36876da8cd22"
-      (reference "ADDR1") (unit 1) (value "74LV165D,118") (footprint "Package_SO:SOIC-16_3.9x9.9mm_P1.27mm")
+      (reference "ADDR1") (unit 1) (value "SN74LV165APWR") (footprint "Package_SO:TSSOP-16_4.4x5mm_P0.65mm")
     )
     (path "/8f6c9fa1-3648-465c-a336-2b2618f99bc1"
-      (reference "ADDR2") (unit 1) (value "74LV165D,118") (footprint "Package_SO:SOIC-16_3.9x9.9mm_P1.27mm")
+      (reference "ADDR2") (unit 1) (value "SN74LV165APWR") (footprint "Package_SO:TSSOP-16_4.4x5mm_P0.65mm")
     )
     (path "/5c84040b-37aa-4dcc-88ef-f10901051605"
-      (reference "ADDR3") (unit 1) (value "74LV165D,118") (footprint "Package_SO:SOIC-16_3.9x9.9mm_P1.27mm")
+      (reference "ADDR3") (unit 1) (value "SN74LV165APWR") (footprint "Package_SO:TSSOP-16_4.4x5mm_P0.65mm")
     )
     (path "/24e56d90-4a27-4fea-a88a-449db4db524c"
-      (reference "ADDR4") (unit 1) (value "74LV165D,118") (footprint "Package_SO:SOIC-16_3.9x9.9mm_P1.27mm")
+      (reference "ADDR4") (unit 1) (value "SN74LV165APWR") (footprint "Package_SO:TSSOP-16_4.4x5mm_P0.65mm")
     )
     (path "/bbdbe439-63b1-44e9-b277-34f4e5557d1a"
